Commit message: Updated urdf

File: src/hexapod/hexapod_description/urdf/hexapod.urdf (robot description, URDF)
Before this commit: robot hexapod, 11 links, 18 joints
Links:
- added link femur_L2, mass 0.2; collision mesh filename=package://hexapod_description/meshes/femur.dae; visual mesh filename=package://hexapod_description/meshes/femur.dae
- added link femur_L3, mass 0.2; collision mesh filename=package://hexapod_description/meshes/femur.dae; visual mesh filename=package://hexapod_description/meshes/femur.dae
- added link femur_R2, mass 0.2; collision mesh filename=package://hexapod_description/meshes/femur.dae; visual mesh filename=package://hexapod_description/meshes/femur.dae
- added link femur_R3, mass 0.2; collision mesh filename=package://hexapod_description/meshes/femur.dae; visual mesh filename=package://hexapod_description/meshes/femur.dae
- added link hip_L1, mass 0.001
- added link hip_L2, mass 0.001
- added link hip_L3, mass 0.001
- added link hip_R1, mass 0.001
- added link hip_R2, mass 0.001
- added link hip_R3, mass 0.001
- added link tibia_L2, mass 0.4; collision mesh filename=package://hexapod_description/meshes/tibia.dae; visual mesh filename=package://hexapod_description/meshes/tibia.dae
- added link tibia_L3, mass 0.4; collision mesh filename=package://hexapod_description/meshes/tibia.dae; visual mesh filename=package://hexapod_description/meshes/tibia.dae
- added link tibia_R2, mass 0.4; collision mesh filename=package://hexapod_description/meshes/tibia.dae; visual mesh filename=package://hexapod_description/meshes/tibia.dae
- added link tibia_R3, mass 0.4; collision mesh filename=package://hexapod_description/meshes/tibia.dae; visual mesh filename=package://hexapod_description/meshes/tibia.dae
- added link world
- link body: mass 0.0 -> 1.0; geometry collision mesh filename=package://hexapod_description/meshes/base.dae; visual mesh filename=package://hexapod_description/meshes/base.dae
- link femur_L1: mass 0.0 -> 0.2; geometry collision mesh filename=package://hexapod_description/meshes/femur.dae; visual mesh filename=package://hexapod_description/meshes/femur.dae
- link femur_R1: mass 0.0 -> 0.2; geometry collision mesh filename=package://hexapod_description/meshes/femur.dae; visual mesh filename=package://hexapod_description/meshes/femur.dae
- link tibia_L1: mass 0.0 -> 0.4; geometry collision mesh filename=package://hexapod_description/meshes/tibia.dae; visual mesh filename=package://hexapod_description/meshes/tibia.dae
- link tibia_R1: mass 0.0 -> 0.4; geometry collision mesh filename=package://hexapod_description/meshes/tibia.dae; visual mesh filename=package://hexapod_description/meshes/tibia.dae
Joints:
- removed joint joint_hip_L1
- removed joint joint_hip_L2
- removed joint joint_hip_L3
- removed joint joint_hip_R1
- removed joint joint_hip_R2
- removed joint joint_hip_R3
- added joint base_joint: type fixed, parent world, child body, origin xyz=0 0 0.5 rpy=0 0 0
- added joint joint_hip1_L1: type revolute, parent body, child hip_L1, origin xyz=-0.02866 0.04964 0.02 rpy=0 0 0, axis 0 0 1, limit lower=-3 upper=3 effort=30.0 velocity=6
- added joint joint_hip1_L2: type revolute, parent body, child hip_L2, origin xyz=-0.05732 0 0.02 rpy=0 0 0, axis 0 0 1, limit lower=-3 upper=3 effort=30.0 velocity=6
- added joint joint_hip1_L3: type revolute, parent body, child hip_L3, origin xyz=-0.02866 -0.04964 0.02 rpy=0 0 0, axis 0 0 1, limit lower=-3 upper=3 effort=30.0 velocity=6
- added joint joint_hip1_R1: type revolute, parent body, child hip_R1, origin xyz=0.02866 0.04964 0.02 rpy=0 0 0, axis 0 0 1, limit lower=-3 upper=3 effort=30.0 velocity=6
- added joint joint_hip1_R2: type revolute, parent body, child hip_R2, origin xyz=0.05732 0 0.02 rpy=0 0 0, axis 0 0 1, limit lower=-3 upper=3 effort=30.0 velocity=6
- added joint joint_hip1_R3: type revolute, parent body, child hip_R3, origin xyz=0.02866 -0.04964 0.02 rpy=0 0 0, axis 0 0 1, limit lower=-3 upper=3 effort=30.0 velocity=6
- added joint joint_hip2_L1: type revolute, parent hip_L1, child femur_L1, origin xyz=0 0 0 rpy=0 0 0, axis 0 1 0, limit lower=-3 upper=3 effort=30.0 velocity=6
- added joint joint_hip2_L2: type revolute, parent hip_L2, child femur_L2, origin xyz=0 0 0 rpy=0 0 0, axis 0 1 0, limit lower=-3 upper=3 effort=30.0 velocity=6
- added joint joint_hip2_L3: type revolute, parent hip_L3, child femur_L3, origin xyz=0 0 0 rpy=0 0 0, axis 0 1 0, limit lower=-3 upper=3 effort=30.0 velocity=6
- added joint joint_hip2_R1: type revolute, parent hip_R1, child femur_R1, origin xyz=0 0 0 rpy=0 0 0, axis 0 1 0, limit lower=-3 upper=3 effort=30.0 velocity=6
- added joint joint_hip2_R2: type revolute, parent hip_R2, child femur_R2, origin xyz=0 0 0 rpy=0 0 0, axis 0 1 0, limit lower=-3 upper=3 effort=30.0 velocity=6
- added joint joint_hip2_R3: type revolute, parent hip_R3, child femur_R3, origin xyz=0 0 0 rpy=0 0 0, axis 0 1 0, limit lower=-3 upper=3 effort=30.0 velocity=6
- joint joint_foot_L1: origin xyz=0.2032 0 0 rpy=0 0 0  -> xyz=0 0 0.08 rpy=0 0 0 
- joint joint_foot_L2: origin xyz=0.2032 0 0 rpy=0 0 0  -> xyz=0 0 0.08 rpy=0 0 0 
- joint joint_foot_L3: origin xyz=0.2032 0 0 rpy=0 0 0  -> xyz=0 0 0.08 rpy=0 0 0 
- joint joint_foot_R1: origin xyz=0.2032 0 0 rpy=0 0 0  -> xyz=0 0 0.08 rpy=0 0 0 
- joint joint_foot_R2: origin xyz=0.2032 0 0 rpy=0 0 0  -> xyz=0 0 0.08 rpy=0 0 0 
- joint joint_foot_R3: origin xyz=0.2032 0 0 rpy=0 0 0  -> xyz=0 0 0.08 rpy=0 0 0 
- joint joint_knee_L1: axis 0 0 1 -> 0 1 0; origin xyz=-0.1016 0.1524 0 rpy=1.57 0 -1.57 -> xyz=0 0 0.04 rpy=0 0 0
- joint joint_knee_L2: axis 0 0 1 -> 0 1 0; origin xyz=-0.1016 0.1524 0 rpy=1.57 0 -1.57 -> xyz=0 0 0.04 rpy=0 0 0
- joint joint_knee_L3: axis 0 0 1 -> 0 1 0; origin xyz=-0.1016 0.1524 0 rpy=1.57 0 -1.57 -> xyz=0 0 0.04 rpy=0 0 0
- joint joint_knee_R1: axis 0 0 1 -> 0 1 0; origin xyz=-0.1016 0.1524 0 rpy=1.57 0 -1.57 -> xyz=0 0 0.04 rpy=0 0 0
- joint joint_knee_R2: axis 0 0 1 -> 0 1 0; origin xyz=-0.1016 0.1524 0 rpy=1.57 0 -1.57 -> xyz=0 0 0.04 rpy=0 0 0
- joint joint_knee_R3: axis 0 0 1 -> 0 1 0; origin xyz=-0.1016 0.1524 0 rpy=1.57 0 -1.57 -> xyz=0 0 0.04 rpy=0 0 0

Commit message: Updated URDF

File: src/hexapod/hexapod_description/urdf/hexapod.urdf (robot description, URDF)
Before this commit: robot hexapod, 26 links, 25 joints
Links:
- link femur_L1: geometry visual mesh filename=package://hexapod_description/meshes/femur.dae
- link femur_L2: geometry visual mesh filename=package://hexapod_description/meshes/femur.dae
- link femur_L3: geometry visual mesh filename=package://hexapod_description/meshes/femur.dae
- link femur_R1: geometry visual mesh filename=package://hexapod_description/meshes/femur.dae
- link femur_R2: geometry visual mesh filename=package://hexapod_description/meshes/femur.dae
- link femur_R3: geometry visual mesh filename=package://hexapod_description/meshes/femur.dae
Joints:
- joint joint_hip1_L1: origin xyz=-0.02866 0.04964 0.02 rpy=0 0 0 -> xyz=0.0 0.0 0.0 rpy=0 0 2.0944
- joint joint_hip1_L2: origin xyz=-0.05732 0 0.02 rpy=0 0 0 -> xyz=0.0 0.0 0.0 rpy=0 0 3.1416
- joint joint_hip1_L3: origin xyz=-0.02866 -0.04964 0.02 rpy=0 0 0 -> xyz=0.0 0.0 0.0 rpy=0 0.5 -2.0944
- joint joint_hip1_R1: origin xyz=0.02866 0.04964 0.02 rpy=0 0 0 -> xyz=0.0 0.0 0.0 rpy=0 0 1.0472
- joint joint_hip1_R2: origin xyz=0.05732 0 0.02 rpy=0 0 0 -> xyz=0.0 0.0 0.0 rpy=0 0 0
- joint joint_hip1_R3: origin xyz=0.02866 -0.04964 0.02 rpy=0 0 0 -> xyz=0.0 0.0 0.0 rpy=0.5 0 -1.0472
- joint joint_knee_L1: axis 0 1 0 -> 0 0 1; origin xyz=0 0 0.04 rpy=0 0 0 -> xyz=0 0 0 rpy=0 0 0
- joint joint_knee_L2: axis 0 1 0 -> 0 0 1; origin xyz=0 0 0.04 rpy=0 0 0 -> xyz=0 0 0 rpy=0 0 0
- joint joint_knee_L3: axis 0 1 0 -> 0 0 1; origin xyz=0 0 0.04 rpy=0 0 0 -> xyz=0 0 0 rpy=0 0 0
- joint joint_knee_R1: axis 0 1 0 -> 0 0 1; origin xyz=0 0 0.04 rpy=0 0 0 -> xyz=0 0 0 rpy=0 0 0
- joint joint_knee_R2: axis 0 1 0 -> 0 0 1; origin xyz=0 0 0.04 rpy=0 0 0 -> xyz=0 0 0 rpy=0 0 0
- joint joint_knee_R3: axis 0 1 0 -> 0 0 1; origin xyz=0 0 0.04 rpy=0 0 0 -> xyz=0 0 0 rpy=0 0 0

Commit message: Updated URDF, working now

File: src/hexapod/hexapod_description/urdf/hexapod.urdf (robot description, URDF)
Before this commit: robot hexapod, 26 links, 25 joints
Joints:
- joint joint_hip1_L1: origin xyz=0.0 0.0 0.0 rpy=0 0 2.0944 -> xyz=-0.02866 0.04964 0.01 rpy=-1.5708 0 0.5236
- joint joint_hip1_L2: origin xyz=0.0 0.0 0.0 rpy=0 0 3.1416 -> xyz=-0.05732 0.0 0.01 rpy=-1.5708 0 1.5708
- joint joint_hip1_L3: origin xyz=0.0 0.0 0.0 rpy=0 0.5 -2.0944 -> xyz=-0.02866 -0.04964 0.01 rpy=-1.5708 0 2.618
- joint joint_hip1_R1: origin xyz=0.0 0.0 0.0 rpy=0 0 1.0472 -> xyz=0.02866 0.04964 0.01 rpy=-1.5708 0 -0.5236
- joint joint_hip1_R2: origin xyz=0.0 0.0 0.0 rpy=0 0 0 -> xyz=0.05732 0.0 0.01 rpy=-1.5708 0 -1.5708
- joint joint_hip1_R3: origin xyz=0.0 0.0 0.0 rpy=0.5 0 -1.0472 -> xyz=0.02866 -0.04964 0.01 rpy=-1.5708 0 -2.618
- joint joint_knee_L1: axis 0 0 1 -> 0 1 0; origin xyz=0 0 0 rpy=0 0 0 -> xyz=0 0 0.04 rpy=-1.5708 0 0
- joint joint_knee_L2: axis 0 0 1 -> 0 1 0; origin xyz=0 0 0 rpy=0 0 0 -> xyz=0 0 0.04 rpy=-1.5708 0 0
- joint joint_knee_L3: axis 0 0 1 -> 0 1 0; origin xyz=0 0 0 rpy=0 0 0 -> xyz=0 0 0.04 rpy=-1.5708 0 0
- joint joint_knee_R1: axis 0 0 1 -> 0 1 0; origin xyz=0 0 0 rpy=0 0 0 -> xyz=0 0 0.04 rpy=-1.5708 0 0
- joint joint_knee_R2: axis 0 0 1 -> 0 1 0; origin xyz=0 0 0 rpy=0 0 0 -> xyz=0 0 0.04 rpy=-1.5708 0 0
- joint joint_knee_R3: axis 0 0 1 -> 0 1 0; origin xyz=0 0 0 rpy=0 0 0 -> xyz=0 0 0.04 rpy=-1.5708 0 0

Commit message: Updated joint axes. Fixed commented out gazebo plugin issue

File: src/hexapod/hexapod_description/urdf/hexapod.urdf (robot description, URDF)
Before this commit: robot hexapod, 26 links, 25 joints
Joints:
- joint joint_hip1_L1: axis 0 0 1 -> 0 1 0
- joint joint_hip1_L2: axis 0 0 1 -> 0 1 0
- joint joint_hip1_L3: axis 0 0 1 -> 0 1 0
- joint joint_hip1_R1: axis 0 0 1 -> 0 1 0
- joint joint_hip1_R2: axis 0 0 1 -> 0 1 0
- joint joint_hip1_R3: axis 0 0 1 -> 0 1 0
- joint joint_hip2_L1: axis 0 1 0 -> 1 0 0
- joint joint_hip2_L2: axis 0 1 0 -> 1 0 0
- joint joint_hip2_L3: axis 0 1 0 -> 1 0 0
- joint joint_hip2_R1: axis 0 1 0 -> 1 0 0
- joint joint_hip2_R2: axis 0 1 0 -> 1 0 0
- joint joint_hip2_R3: axis 0 1 0 -> 1 0 0
- joint joint_knee_L1: axis 0 1 0 -> 1 0 0
- joint joint_knee_L2: axis 0 1 0 -> 1 0 0
- joint joint_knee_L3: axis 0 1 0 -> 1 0 0
- joint joint_knee_R1: axis 0 1 0 -> 1 0 0
- joint joint_knee_R2: axis 0 1 0 -> 1 0 0
- joint joint_knee_R3: axis 0 1 0 -> 1 0 0

Commit message: Updated URDF with temporary inertia values to avoid Gazebo jitter bug

File: src/hexapod/hexapod_description/urdf/hexapod.urdf (robot description, URDF)
Before this commit: robot hexapod, 26 links, 25 joints
Links:
- removed link hip_L1
- removed link hip_L2
- removed link hip_L3
- removed link hip_R1
- removed link hip_R2
- removed link hip_R3
- added link coxa_L1, mass 0.1; visual mesh filename=package://hexapod_description/meshes/coxa.dae
- added link coxa_L2, mass 0.1; visual mesh filename=package://hexapod_description/meshes/coxa.dae
- added link coxa_L3, mass 0.1; visual mesh filename=package://hexapod_description/meshes/coxa.dae
- added link coxa_R1, mass 0.1; visual mesh filename=package://hexapod_description/meshes/coxa.dae
- added link coxa_R2, mass 0.1; visual mesh filename=package://hexapod_description/meshes/coxa.dae
- added link coxa_R3, mass 0.1; visual mesh filename=package://hexapod_description/meshes/coxa.dae
- link body: mass 1.0 -> 2.0
- link femur_L1: mass 0.2 -> 0.4
- link femur_L2: mass 0.2 -> 0.4
- link femur_L3: mass 0.2 -> 0.4
- link femur_R1: mass 0.2 -> 0.4
- link femur_R2: mass 0.2 -> 0.4
- link femur_R3: mass 0.2 -> 0.4
- link tibia_L1: mass 0.4 -> 0.8
- link tibia_L2: mass 0.4 -> 0.8
- link tibia_L3: mass 0.4 -> 0.8
- link tibia_R1: mass 0.4 -> 0.8
- link tibia_R2: mass 0.4 -> 0.8
- link tibia_R3: mass 0.4 -> 0.8
Joints:
- joint base_joint: origin xyz=0 0 0.5 rpy=0 0 0 -> xyz=0 0 0.3 rpy=0 0 0
- joint joint_hip1_L1: child hip_L1 -> coxa_L1
- joint joint_hip1_L2: child hip_L2 -> coxa_L2
- joint joint_hip1_L3: child hip_L3 -> coxa_L3
- joint joint_hip1_R1: child hip_R1 -> coxa_R1
- joint joint_hip1_R2: child hip_R2 -> coxa_R2
- joint joint_hip1_R3: child hip_R3 -> coxa_R3
- joint joint_hip2_L1: origin xyz=0 0 0 rpy=0 0 0 -> xyz=0 0 0.01 rpy=0 0 0; parent hip_L1 -> coxa_L1
- joint joint_hip2_L2: origin xyz=0 0 0 rpy=0 0 0 -> xyz=0 0 0.01 rpy=0 0 0; parent hip_L2 -> coxa_L2
- joint joint_hip2_L3: origin xyz=0 0 0 rpy=0 0 0 -> xyz=0 0 0.01 rpy=0 0 0; parent hip_L3 -> coxa_L3
- joint joint_hip2_R1: origin xyz=0 0 0 rpy=0 0 0 -> xyz=0 0 0.01 rpy=0 0 0; parent hip_R1 -> coxa_R1
- joint joint_hip2_R2: origin xyz=0 0 0 rpy=0 0 0 -> xyz=0 0 0.01 rpy=0 0 0; parent hip_R2 -> coxa_R2
- joint joint_hip2_R3: origin xyz=0 0 0 rpy=0 0 0 -> xyz=0 0 0.01 rpy=0 0 0; parent hip_R3 -> coxa_R3

Commit message: Updated URDF and gazebo to fit new model

File: src/hexapod/hexapod_description/urdf/hexapod.urdf (robot description, URDF)
Before this commit: robot hexapod, 26 links, 25 joints
Links:
- removed link world
- link body: geometry collision mesh filename=package://hexapod_description/meshes/base_v2.dae; visual mesh filename=package://hexapod_description/meshes/base_v2.dae
Joints:
- removed joint base_joint
- joint joint_hip1_L1: origin xyz=-0.02866 0.04964 0.01 rpy=-1.5708 0 0.5236 -> xyz=-0.04 0.06928 0.01 rpy=-1.5708 0 0.5
- joint joint_hip1_L2: origin xyz=-0.05732 0.0 0.01 rpy=-1.5708 0 1.5708 -> xyz=-0.080 0.0 0.01 rpy=-1.5708 0 1.5708
- joint joint_hip1_L3: origin xyz=-0.02866 -0.04964 0.01 rpy=-1.5708 0 2.618 -> xyz=-0.04 -0.06928 0.01 rpy=-1.5708 0 2.6416
- joint joint_hip1_R1: origin xyz=0.02866 0.04964 0.01 rpy=-1.5708 0 -0.5236 -> xyz=0.04 0.06928 0.01 rpy=-1.5708 0 -0.5
- joint joint_hip1_R2: origin xyz=0.05732 0.0 0.01 rpy=-1.5708 0 -1.5708 -> xyz=0.080 0.0 0.01 rpy=-1.5708 0 -1.5708
- joint joint_hip1_R3: origin xyz=0.02866 -0.04964 0.01 rpy=-1.5708 0 -2.618 -> xyz=0.04 -0.06928 0.01 rpy=-1.5708 0 -2.6416
- joint joint_knee_L1: origin xyz=0 0 0.04 rpy=-1.5708 0 0 -> xyz=0 0 0.04 rpy=0 0 0
- joint joint_knee_L2: origin xyz=0 0 0.04 rpy=-1.5708 0 0 -> xyz=0 0 0.04 rpy=0 0 0
- joint joint_knee_L3: origin xyz=0 0 0.04 rpy=-1.5708 0 0 -> xyz=0 0 0.04 rpy=0 0 0
- joint joint_knee_R1: origin xyz=0 0 0.04 rpy=-1.5708 0 0 -> xyz=0 0 0.04 rpy=0 0 0
- joint joint_knee_R2: origin xyz=0 0 0.04 rpy=-1.5708 0 0 -> xyz=0 0 0.04 rpy=0 0 0
- joint joint_knee_R3: origin xyz=0 0 0.04 rpy=-1.5708 0 0 -> xyz=0 0 0.04 rpy=0 0 0
