Commit message: Updated ankle joint direction

File: src/hexapod/hexapod_description/urdf/hexapod.urdf.xacro (robot description, xacro)
@@ -119,5 +119,5 @@
             <parent link="${robot_name}/${prefix}_femur_link"/>
             <child link="${robot_name}/${prefix}_tibia_link"/>
-            <axis xyz="1 0 0"/>
+            <axis xyz="-1 0 0"/>
             <limit lower="0" upper="${2*pi/3}" effort="30" velocity="${pi}"/>
             <safety_controller k_position="100.0" k_velocity="40.0" soft_lower_limit="-3" soft_upper_limit="3"/>

Commit message: Fixed roll pitch yaw order

File: src/hexapod/hexapod_description/urdf/hexapod.urdf.xacro (robot description, xacro)
@@ -38,5 +38,5 @@
     </xacro:macro>
     <!-- ============================ Leg Macro ============================ -->
-    <xacro:macro name="leg" params="prefix x y z pitch roll yaw">
+    <xacro:macro name="leg" params="prefix x y z roll pitch yaw">
         <!-- Links -->
         <link name="${robot_name}/${prefix}_coxa_link">
@@ -100,5 +100,5 @@
         <!-- Joints -->
         <joint name="${prefix}_hip_joint" type="revolute">
-            <origin xyz="${x} ${y} ${z}" rpy="${pitch} ${roll} ${yaw}"/>
+            <origin xyz="${x} ${y} ${z}" rpy="${roll} ${pitch} ${yaw}"/>
             <parent link="${robot_name}/base_link"/>
             <child link="${robot_name}/${prefix}_coxa_link"/>
@@ -203,25 +203,25 @@
     <xacro:leg prefix="L1"
         x="${base_radius*cos(L1_angle)}" y="${base_radius*sin(L1_angle)}" z="0.01"
-        pitch="${-pi/2}" roll="0" yaw="0.5"
+        roll="${-pi/2}" pitch="0.0" yaw="0.5"
     />
     <xacro:leg prefix="R1"
         x="${base_radius*cos(R1_angle)}" y="${base_radius*sin(R1_angle)}" z="0.01"
-        pitch="${-pi/2}" roll="0" yaw="-0.5"
+        roll="${-pi/2}" pitch="0.0" yaw="-0.5"
     />
     <xacro:leg prefix="L2"
         x="${base_radius*cos(L2_angle)}" y="${base_radius*sin(L2_angle)}" z="0.01"
-        pitch="${-pi/2}" roll="0" yaw="${pi/2}"
+        roll="${-pi/2}" pitch="0.0" yaw="${pi/2}"
     />
     <xacro:leg prefix="R2"
         x="${base_radius*cos(R2_angle)}" y="${base_radius*sin(R2_angle)}" z="0.01"
-        pitch="${-pi/2}" roll="0" yaw="${-pi/2}"
+        roll="${-pi/2}" pitch="0.0" yaw="${-pi/2}"
     />
     <xacro:leg prefix="L3"
         x="${base_radius*cos(L3_angle)}" y="${base_radius*sin(L3_angle)}" z="0.01"
-        pitch="${-pi/2}" roll="0" yaw="${pi-0.5}"
+        roll="${-pi/2}" pitch="0.0" yaw="${pi-0.5}"
     />
     <xacro:leg prefix="R3"
         x="${base_radius*cos(R3_angle)}" y="${base_radius*sin(R3_angle)}" z="0.01"
-        pitch="${-pi/2}" roll="0" yaw="${-(pi-0.5)}"
+        roll="${-pi/2}" pitch="0.0" yaw="${-(pi-0.5)}"
     />
     <!-- ============================= Gazebo ============================= -->

Commit message: Fixed direction of hip joint polarity

File: src/hexapod/hexapod_description/urdf/hexapod.urdf.xacro (robot description, xacro)
@@ -103,5 +103,5 @@
             <parent link="${robot_name}/base_link"/>
             <child link="${robot_name}/${prefix}_coxa_link"/>
-            <axis xyz="0 1 0"/>
+            <axis xyz="0 -1 0"/>
             <limit lower="${-pi/2}" upper="${pi/2}" effort="30" velocity="${pi}"/>
             <safety_controller k_position="100.0" k_velocity="40.0" soft_lower_limit="-3" soft_upper_limit="3"/>

Commit message: Changed implementation to publish values that can be changed on the fly and send only a few as part of the gait goal

File: src/hexapod/hexapod_description/urdf/hexapod.urdf.xacro (robot description, xacro)
@@ -188,10 +188,10 @@
     </xacro:macro>
     <!-- ========================== Generate URDF ========================== -->
-    <!-- <link name="world"/>
-        <joint name="fixed_joint" type="fixed">
-            <origin xyz="0 0 0.3" rpy="0 0 0"/>
-            <parent link="world"/>
-            <child link="dummy_link"/>
-        </joint> -->
+    <link name="world"/>
+    <joint name="fixed_joint" type="fixed">
+        <origin xyz="0 0 0.3" rpy="0 0 0"/>
+        <parent link="world"/>
+        <child link="dummy_link"/>
+    </joint>
     <!-- Dummy Link and Joint avoids "KDL does not support a root link with an inertia" error -->
     <link name="dummy_link"/>

Commit message: Fixed Walk() and Rotate() functions. Ramp down still weird

File: src/hexapod/hexapod_description/urdf/hexapod.urdf.xacro (robot description, xacro)
@@ -188,10 +188,10 @@
     </xacro:macro>
     <!-- ========================== Generate URDF ========================== -->
-    <link name="world"/>
+    <!-- <link name="world"/>
     <joint name="fixed_joint" type="fixed">
         <origin xyz="0 0 0.3" rpy="0 0 0"/>
         <parent link="world"/>
         <child link="dummy_link"/>
-    </joint>
+    </joint> -->
     <!-- Dummy Link and Joint avoids "KDL does not support a root link with an inertia" error -->
     <link name="dummy_link"/>

Commit message: Added option to make foot use revolute joint. Not being used now

File: src/hexapod/hexapod_description/urdf/hexapod.urdf.xacro (robot description, xacro)
@@ -11,4 +11,5 @@
     <xacro:property name="femur_mass"   value="0.4"/>
     <xacro:property name="tibia_mass"   value="0.8"/>
+    <!-- <xacro:property name="foot_mass"    value="0.01"/> -->
     <xacro:property name="inertia"      value="0.1"/>
     <xacro:property name="L1_angle"     value="${2*pi/3}"/>
@@ -98,4 +99,11 @@
         </link>
         <link name="${robot_name}/${prefix}_foot_link"/>
+        <!-- <link name="${robot_name}/${prefix}_foot_link">
+            <inertial>
+                <origin xyz="0 0 0" rpy="0 0 0"/>
+                <mass value="${foot_mass}"/>
+                <inertia ixx="${inertia}" iyy="${inertia}" izz="${inertia}" ixy="0.0" ixz="0.0" iyz="0.0"/>
+            </inertial>
+        </link> -->
         <!-- Joints -->
         <joint name="${prefix}_hip_joint" type="revolute">
@@ -128,4 +136,12 @@
             <child link="${robot_name}/${prefix}_foot_link"/>
         </joint>
+        <!-- <joint name="${prefix}_foot_joint" type="revolute">
+            <origin xyz="0 0 ${tibia_length}" rpy="0 0 0"/>
+            <parent link="${robot_name}/${prefix}_tibia_link"/>
+            <child link="${robot_name}/${prefix}_foot_link"/>
+            <axis xyz="0 0 1"/>
+            <limit lower="0" upper="0" effort="30" velocity="0"/>
+            <safety_controller k_position="100.0" k_velocity="40.0" soft_lower_limit="-3" soft_upper_limit="3"/>
+        </joint> -->
         <!-- Gazebo Collision -->
         <gazebo reference="${prefix}_tibia_link">

Commit message: Added joint limit xacro properties. Currently widened limits but need to make more realistic later

File: src/hexapod/hexapod_description/urdf/hexapod.urdf.xacro (robot description, xacro)
@@ -2,21 +2,33 @@
 <robot name="hexapod" xmlns:xacro="http://www.ros.org/wiki/xacro">
     <!-- ============================ Constants ============================ -->
-    <xacro:property name="robot_name"   value="hexapod"/>
-    <xacro:property name="base_radius"  value="0.08"/>
-    <xacro:property name="coxa_length"  value="0.01"/>
-    <xacro:property name="femur_length" value="0.04"/>
-    <xacro:property name="tibia_length" value="0.08"/>
-    <xacro:property name="base_mass"    value="2.0"/>
-    <xacro:property name="coxa_mass"    value="0.1"/>
-    <xacro:property name="femur_mass"   value="0.4"/>
-    <xacro:property name="tibia_mass"   value="0.8"/>
+    <xacro:property name="robot_name"           value="hexapod"/>
+    <xacro:property name="base_radius"          value="0.08"/>
+    <xacro:property name="coxa_length"          value="0.01"/>
+    <xacro:property name="femur_length"         value="0.04"/>
+    <xacro:property name="tibia_length"         value="0.08"/>
+    <xacro:property name="base_mass"            value="2.0"/>
+    <xacro:property name="coxa_mass"            value="0.1"/>
+    <xacro:property name="femur_mass"           value="0.4"/>
+    <xacro:property name="tibia_mass"           value="0.8"/>
     <!-- <xacro:property name="foot_mass"    value="0.01"/> -->
-    <xacro:property name="inertia"      value="0.1"/>
-    <xacro:property name="L1_angle"     value="${2*pi/3}"/>
-    <xacro:property name="R1_angle"     value="${pi/3}"/>
-    <xacro:property name="L2_angle"     value="${pi}"/>
-    <xacro:property name="R2_angle"     value="${0}"/>
-    <xacro:property name="L3_angle"     value="${4*pi/3}"/>
-    <xacro:property name="R3_angle"     value="${5*pi/3}"/>
+    <xacro:property name="inertia"              value="0.1"/>
+    <xacro:property name="L1_angle"             value="${2*pi/3}"/>
+    <xacro:property name="R1_angle"             value="${pi/3}"/>
+    <xacro:property name="L2_angle"             value="${pi}"/>
+    <xacro:property name="R2_angle"             value="${0}"/>
+    <xacro:property name="L3_angle"             value="${4*pi/3}"/>
+    <xacro:property name="R3_angle"             value="${5*pi/3}"/>
+    <!-- <xacro:property name="hip_lower_limit"      value="${-pi/2}"/>
+    <xacro:property name="hip_upper_limit"      value="${pi/2}"/>
+    <xacro:property name="knee_lower_limit"     value="${-pi/6}"/>
+    <xacro:property name="knee_upper_limit"     value="${pi/2}"/>
+    <xacro:property name="ankle_lower_limit"    value="${0}"/>
+    <xacro:property name="ankle_upper_limit"    value="${2*pi/3}"/> -->
+    <xacro:property name="hip_lower_limit"      value="${-pi}"/>
+    <xacro:property name="hip_upper_limit"      value="${pi}"/>
+    <xacro:property name="knee_lower_limit"     value="${-pi/2}"/>
+    <xacro:property name="knee_upper_limit"     value="${pi/2}"/>
+    <xacro:property name="ankle_lower_limit"    value="${0}"/>
+    <xacro:property name="ankle_upper_limit"    value="${pi}"/>
     <!-- =========================== Base Macro =========================== -->
     <xacro:macro name="base">
@@ -112,5 +124,5 @@
             <child link="${robot_name}/${prefix}_coxa_link"/>
             <axis xyz="0 -1 0"/>
-            <limit lower="${-pi/2}" upper="${pi/2}" effort="30" velocity="${pi}"/>
+            <limit lower="${hip_lower_limit}" upper="${hip_upper_limit}" effort="30" velocity="${pi}"/>
             <safety_controller k_position="100.0" k_velocity="40.0" soft_lower_limit="-3" soft_upper_limit="3"/>
         </joint>
@@ -120,5 +132,5 @@
             <child link="${robot_name}/${prefix}_femur_link"/>
             <axis xyz="1 0 0"/>
-            <limit lower="${-pi/6}" upper="${pi/2}" effort="30" velocity="${pi}"/>
+            <limit lower="${knee_lower_limit}" upper="${knee_upper_limit}" effort="30" velocity="${pi}"/>
             <safety_controller k_position="100.0" k_velocity="40.0" soft_lower_limit="-3" soft_upper_limit="3"/>
         </joint>
@@ -128,5 +140,5 @@
             <child link="${robot_name}/${prefix}_tibia_link"/>
             <axis xyz="-1 0 0"/>
-            <limit lower="0" upper="${2*pi/3}" effort="30" velocity="${pi}"/>
+            <limit lower="${ankle_lower_limit}" upper="${ankle_upper_limit}" effort="30" velocity="${pi}"/>
             <safety_controller k_position="100.0" k_velocity="40.0" soft_lower_limit="-3" soft_upper_limit="3"/>
         </joint>
@@ -204,10 +216,10 @@
     </xacro:macro>
     <!-- ========================== Generate URDF ========================== -->
-    <!-- <link name="world"/>
+    <link name="world"/>
     <joint name="fixed_joint" type="fixed">
         <origin xyz="0 0 0.3" rpy="0 0 0"/>
         <parent link="world"/>
         <child link="dummy_link"/>
-    </joint> -->
+    </joint>
     <!-- Dummy Link and Joint avoids "KDL does not support a root link with an inertia" error -->
     <link name="dummy_link"/>

Commit message: Added src/unused for bookkeeping

File: src/hexapod/hexapod_description/urdf/hexapod.urdf.xacro (robot description, xacro)
@@ -216,10 +216,11 @@
     </xacro:macro>
     <!-- ========================== Generate URDF ========================== -->
-    <link name="world"/>
+    <!-- Uncomment out the below code to position the robot in midair -->
+    <!-- <link name="world"/>
     <joint name="fixed_joint" type="fixed">
         <origin xyz="0 0 0.3" rpy="0 0 0"/>
         <parent link="world"/>
         <child link="dummy_link"/>
-    </joint>
+    </joint> -->
     <!-- Dummy Link and Joint avoids "KDL does not support a root link with an inertia" error -->
     <link name="dummy_link"/>

Commit message: Increased mass of each section

File: src/hexapod/hexapod_description/urdf/hexapod.urdf.xacro (robot description, xacro)
@@ -7,8 +7,8 @@
     <xacro:property name="femur_length"         value="0.04"/>
     <xacro:property name="tibia_length"         value="0.08"/>
-    <xacro:property name="base_mass"            value="2.0"/>
-    <xacro:property name="coxa_mass"            value="0.1"/>
-    <xacro:property name="femur_mass"           value="0.4"/>
-    <xacro:property name="tibia_mass"           value="0.8"/>
+    <xacro:property name="base_mass"            value="4.0"/>
+    <xacro:property name="coxa_mass"            value="0.2"/>
+    <xacro:property name="femur_mass"           value="0.8"/>
+    <xacro:property name="tibia_mass"           value="1.6"/>
     <!-- <xacro:property name="foot_mass"    value="0.01"/> -->
     <xacro:property name="inertia"              value="0.1"/>

Commit message: Added depth camera to urdf.xacro

File: src/hexapod/hexapod_description/urdf/hexapod.urdf.xacro (robot description, xacro)
@@ -4,4 +4,5 @@
     <xacro:property name="robot_name"           value="hexapod"/>
     <xacro:property name="base_radius"          value="0.08"/>
+    <xacro:property name="base_depth"           value="0.02"/>
     <xacro:property name="coxa_length"          value="0.01"/>
     <xacro:property name="femur_length"         value="0.04"/>
@@ -31,4 +32,6 @@
     <xacro:property name="ankle_lower_limit"    value="${0}"/>
     <xacro:property name="ankle_upper_limit"    value="${pi}"/>
+    <xacro:property name="camera_name"          value="depth_camera"/>
+    <xacro:property name="camera_size"          value="0.02" />
     <!-- =========================== Base Macro =========================== -->
     <xacro:macro name="base">
@@ -254,8 +257,124 @@
         roll="${-pi/2}" pitch="0.0" yaw="${-(pi-0.5)}"
     />
+    <!-- ============================= Camera ============================== -->
+    <joint name="camera_joint" type="fixed">
+        <axis xyz="0 0 1" />
+        <origin xyz="0 ${base_radius - camera_size/2} ${base_depth + camera_size/2}"
+                rpy="0 0 ${pi/2}"/>
+        <parent link="${robot_name}/base_link"/>
+        <child link="depth_camera_link"/>
+    </joint>
+    <!-- Depth Camera -->
+    <link name="depth_camera_link">
+        <collision>
+            <origin xyz="0 0 0" rpy="0 0 0"/>
+            <geometry>
+                <box size="${camera_size} ${camera_size} ${camera_size}"/>
+            </geometry>
+        </collision>
+        <visual>
+            <origin xyz="0 0 0" rpy="0 0 0"/>
+            <geometry>
+                <box size="${camera_size} ${camera_size} ${camera_size}"/>
+            </geometry>
+        </visual>
+        <inertial>
+            <mass value="1e-5" />
+            <origin xyz="0 0 0" rpy="0 0 0"/>
+            <inertia ixx="1e-6" ixy="0" ixz="0" iyy="1e-6" iyz="0" izz="1e-6" />
+        </inertial>
+    </link>
     <!-- ============================= Gazebo ============================= -->
+    <!-- ROS control -->
     <gazebo>
-        <!-- IMU, not used yet -->
-        <!-- <plugin name="imu_plugin" filename="libgazebo_ros_imu.so">
+        <plugin name="gazebo_ros_control" filename="libgazebo_ros_control.so">
+            <robotNamespace>/hexapod</robotNamespace>
+        </plugin>
+    </gazebo>
+    <gazebo reference="depth_camera_link">
+        <material>Gazebo/Grey</material>
+    </gazebo>
+    <!-- Depth Camera -->
+    <gazebo reference="depth_camera_link">
+        <sensor name="depth_camera" type="depth">
+            <update_rate>20.0</update_rate>
+            <camera>
+                <horizontal_fov>1.047198</horizontal_fov>
+                <image>
+                    <width>640</width>
+                    <height>480</height>
+                    <format>R8G8B8</format>
+                </image>
+                <clip>
+                    <near>0.01</near>
+                    <far>3.0</far>
+                </clip>
+            </camera>
+            <plugin name="depth_camera_controller" filename="libgazebo_ros_openni_kinect.so">
+                <baseline>0.2</baseline>
+                <alwaysOn>true</alwaysOn>
+                <updateRate>0.0</updateRate>
+                <cameraName>camera_ir</cameraName>
+                <imageTopicName>/camera/color/image_raw</imageTopicName>
+                <cameraInfoTopicName>/camera/color/camera_info</cameraInfoTopicName>
+                <depthImageTopicName>/camera/depth/image_raw</depthImageTopicName>
+                <depthImageInfoTopicName>/camera/depth/camera_info</depthImageInfoTopicName>
+                <pointCloudTopicName>/camera/depth/points</pointCloudTopicName>
+                <frameName>depth_camera_link</frameName>
+                <pointCloudCutoff>0.01</pointCloudCutoff>
+                <pointCloudCutoffMax>3.0</pointCloudCutoffMax>
+                <distortionK1>0</distortionK1>
+                <distortionK2>0</distortionK2>
+                <distortionK3>0</distortionK3>
+                <distortionT1>0</distortionT1>
+                <distortionT2>0</distortionT2>
+                <CxPrime>0</CxPrime>
+                <Cx>0</Cx>
+                <Cy>0</Cy>
+                <focalLength>0</focalLength>
+                <hackBaseline>0</hackBaseline>
+            </plugin>
+        </sensor>
+    </gazebo>
+    <!-- Camera -->
+    <!-- <gazebo reference="camera_link">
+        <sensor type="camera" name="camera1">
+        <update_rate>30.0</update_rate>
+        <camera name="camera">
+            <horizontal_fov>1.3962634</horizontal_fov>
+            <image>
+            <width>800</width>
+            <height>800</height>
+            <format>R8G8B8</format>
+            </image>
+            <clip>
+            <near>0.02</near>
+            <far>300</far>
+            </clip>
+            <noise>
+            <type>gaussian</type>
+            <mean>0.0</mean>
+            <stddev>0.007</stddev>
+            </noise>
+        </camera>
+        <plugin name="camera_controller" filename="libgazebo_ros_camera.so">
+            <alwaysOn>true</alwaysOn>
+            <updateRate>0.0</updateRate>
+            <cameraName>camera</cameraName>
+            <imageTopicName>image_raw</imageTopicName>
+            <cameraInfoTopicName>camera_info</cameraInfoTopicName>
+            <frameName>camera_link</frameName>
+            <hackBaseline>0.07</hackBaseline>
+            <distortionK1>0.0</distortionK1>
+            <distortionK2>0.0</distortionK2>
+            <distortionK3>0.0</distortionK3>
+            <distortionT1>0.0</distortionT1>
+            <distortionT2>0.0</distortionT2>
+        </plugin>
+        </sensor>
+    </gazebo> -->
+    <!-- IMU, not used yet -->
+    <!-- <gazebo reference="IMU_link">
+        <plugin name="imu_plugin" filename="libgazebo_ros_imu.so">
             <alwaysOn>true</alwaysOn>
             <bodyName>body</bodyName>
@@ -264,8 +383,5 @@
             <gaussianNoise>0.0</gaussianNoise>
             <updateRate>40.0</updateRate>
-        </plugin> -->
-        <plugin name="gazebo_ros_control" filename="libgazebo_ros_control.so">
-            <robotNamespace>/hexapod</robotNamespace>
         </plugin>
-    </gazebo>
+    </gazebo> -->
 </robot>
